File: src/name-card.kicad_sch (KiCad schematic)
At the start: 12 parts, among them J1 AVR-ISP-6, SW1 SW_Push, U1 ATtiny25V-10S

Commit message: Add PCB
Parts:
- added AE1: Antenna_Loop, Library:NFC Coil, symbol Device:Antenna_Loop
- added C3: 0.1uF, Capacitor_SMD:C_0402_1005Metric, symbol Device:C
- added U2: ST25DV64K-JFR6D3, Package_DFN_QFN:ST_UFDFPN-12-1EP_3x3mm_P0.5mm_EP1.4x2.55mm, symbol RF_NFC:ST25DV64K-JFR6D3
- J1: LCSC C65114 -> (none); now left out of the parts list
Connections:
- net +3.3V: now also C3.1, U2.10 (VDCG), U2.12 (VCC)
- net GND: now also C3.2, U2.6 (VSS)
- new net: AE1.1, U2.4 (AC0)
- new net: AE1.2, U2.5 (AC1)
- no-connect marks 0 -> 5
